File: 00-produccion-pcbs/1-versiones-profes/grupo-01/g-01-pie-01-rev-a/g-01-pie-01-rev-a.kicad_pcb (KiCad board)
At the start: 2 copper layers, 94.6 x 75.6 mm, 48 parts, among them J2 Conn_01x02_Pin, J4 Barrel_Jack_Switch, J5 Barrel_Jack_Switch, J6 AudioJack2_SwitchT, J7 Conn_01x03_Pin, Q1 2N2222, SW3 SW_SPDT, U1 NE555P, U3 L7805, U4 TL072

Commit message: agregar archivos g01-01
Parts:
- added J8: AudioJack2_SwitchT, dis8644:PJ301M-12, F.Cu at (118.0, 114.5)
- added J9: AudioJack2_SwitchT, dis8644:PJ301M-12, F.Cu at (174.6, 115.0)
- added R7: 1k, Resistor_THT:R_Axial_DIN0207_L6.3mm_D2.5mm_P10.16mm_Horizontal, B.Cu at (154.5, 86.4)
- added R8: 1k, Resistor_THT:R_Axial_DIN0207_L6.3mm_D2.5mm_P10.16mm_Horizontal, B.Cu at (128.9, 113.2)
- C12: value 4.7n -> 4n7
- C2, C3: value 100 u -> 100u
- Q1: footprint Package_TO_SOT_THT:TO-39-3 -> Package_TO_SOT_THT:TO-92_Inline_Wide
- R15: value 20k -> 2M
- moved J4 11.7 mm to (113.0, 88.8), turned to 0 degrees
- moved J5 10.8 mm to (180.0, 91.0), turned to 180 degrees
- moved Q1 8.98 mm to (124.5, 119.0)
- moved R5 4.99 mm to (169.3, 121.5)
- moved C2 4.00 mm to (133.2, 116.5)
- moved C12 2.35 mm to (157.9, 80.0), turned to 90 degrees
Connections:
- C9 pad 1: Net-(J2-Pin_1) -> Net-(C9-Pad1)
- J6 pad 1: Net-(D2-A) -> Net-(J6-Pad1)
- J6 pad 2: Net-(D2-A) -> Net-(J6-Pad1)
- R15 pad 1: Net-(J2-Pin_1) -> Net-(C9-Pad1)
Routing:
- net Net-(J9-Pad3): track 0.00 -> 47.9 mm, vias 0 -> 3
- net Net-(J2-Pin_1): track 38.4 -> 0.00 mm
- net Net-(C9-Pad1): track 0.00 -> 31.4 mm
- net Net-(D2-A): track 99.6 -> 71.7 mm, vias 6 -> 5
- net Net-(J6-Pad1): track 0.00 -> 25.5 mm
- net Net-(SW3-A): track 109.0 -> 88.0 mm
- net VBUS: track 163.1 -> 179.1 mm
- net Net-(D1-A): track 53.6 -> 65.7 mm
- net Net-(Q1-C): track 30.2 -> 21.7 mm
- net Net-(Q1-B): track 27.4 -> 33.5 mm, vias 0 -> 1
- net Net-(U1-DISCH): track 60.1 -> 54.7 mm
- net +5V: track 267.7 -> 272.8 mm
