File: 00-produccion-pcbs/1-versiones-profes/grupo-01/g-01-pie-01-rev-a/g-01-pie-01-rev-a.kicad_sch (KiCad schematic)
At the start: 48 parts, among them J2 Conn_01x02_Pin, J4 Barrel_Jack_Switch, J5 Barrel_Jack_Switch, J6 AudioJack2_SwitchT, J7 Conn_01x03_Pin, Q1 2N2222, SW3 SW_SPDT, U1 NE555P, U3 L7805, U4 TL072

Commit message: agregar archivos g01-01
Parts:
- removed J2: Conn_01x02_Pin, Connector_PinSocket_2.54mm:PinSocket_1x02_P2.54mm_Vertical, symbol Connector:Conn_01x02_Pin
- added J8, J9: AudioJack2_SwitchT, dis8644:PJ301M-12, symbol Connector_Audio:AudioJack2_SwitchT
- added R7, R8: 1k, Resistor_THT:R_Axial_DIN0207_L6.3mm_D2.5mm_P10.16mm_Horizontal, symbol Device:R
- C12: value 4.7n -> 4n7
- C2, C3: value 100 u -> 100u
- R15: value 20k -> 2M
Connections:
- net GND: now also J9.1
- net VBUS: now also J8.1
- net at C1.1, C12.1, D1.2 (A)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: now also R8.1
- net at C9.1, R15.1: now also J8.3
- net at D2.2 (A), U1.3 (OUT): now also R7.1; no longer J6.1, J6.2
- new net: J9.3, R8.2
- new net: J6.1, J6.2, R7.2
